File: hardware/cm-conn2.kicad_sch (KiCad schematic)
At the start: 1 part

Commit message: feat: add InvenTree IPN field to all schematic symbols
102 components mapped to 41 unique InvenTree part numbers.
IPN format: category prefix + sequential number (e.g. C-001, R-002, U-009).
Parts:
- CM1: IPN (none) -> J-002
Changed lines of the file:
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@@
+			)
+		)
+		(property "IPN" "J-002"
+			(at 0 0 0)
+			(show_name no)
+			(do_not_autoplace no)
+			(hide yes)
+			(effects
+				(font
+					(size 1.27 1.27)
+				)
 			)
 		)
