File: hardware/cm-conn2.kicad_sch (KiCad schematic)
At the start: 1 part

Commit message: chore: remove redundant supplier fields, keep IPN as single link to InvenTree
Removed: Supplier, Digikey, Notes, KiLib_Generator, Mouser, Arrow fields.
InvenTree IPN is now the only external reference in the schematic.
Parts:
- CM1: Notes DF40C-100DS-0.4V(51) -> (none); Supplier https://www.digikey.ch/de/products/detail/hirose-electric-c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 -> (none)
Changed lines of the file:
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@@
 			)
 		)
-		(property "Notes" "DF40C-100DS-0.4V(51)"
-			(at -50.8 104.14 0)
+		(property "IPN" "J-002"
+			(at 0 0 0)
 			(hide yes)
 			(show_name no)
@@
 			(effects
 				(font
-					(size 1.27 1.27)
-				)
-			)
-		)
-		(property "Supplier" "https://www.digikey.ch/de/products/detail/hirose-electric-co-ltd/DF40C-100DS-0-4V-51/1969476"
-			(at -50.8 104.14 0)
-			(hide yes)
-			(show_name no)
-			(do_not_autoplace no)
-			(effects
-				(font
-					(size 1.27 1.27)
-				)
-			)
-		)
-		(property "IPN" "J-002"
-			(at 0 0 0)
-			(show_name no)
-			(do_not_autoplace no)
-			(hide yes)
-			(effects
-				(font
