File: hardware/psu.kicad_sch (KiCad schematic)
At the start: 36 parts, among them J6 12V Screw Terminal, J7 12V Barrel, Q6 FDS4435BZ, U6 NCP1117-3.3_SOT223, U7 AP64501SP-13

Commit message: feat: add InvenTree IPN field to all schematic symbols
102 components mapped to 41 unique InvenTree part numbers.
IPN format: category prefix + sequential number (e.g. C-001, R-002, U-009).
Parts:
- C25, C29, C30, C32, C33, C34, C35, C36, C39, C40, C41, C42, C43, C44, C46: IPN (none) -> C-003
- C26: IPN (none) -> C-020
- C27: IPN (none) -> C-005
- C28, C45: IPN (none) -> C-001
- C31, C37: IPN (none) -> C-004
- C38: IPN (none) -> C-006
- F1: IPN (none) -> F-002
- J7: IPN (none) -> J-001
- L1: IPN (none) -> L-001
- Q6: IPN (none) -> Q-001
- R24: IPN (none) -> R-005
- R25: IPN (none) -> R-006
- R26: IPN (none) -> R-007
- R27: IPN (none) -> R-001
- U6: IPN (none) -> U-002
- U7: IPN (none) -> U-001

Commit message: chore: remove redundant supplier fields, keep IPN as single link to InvenTree
Removed: Supplier, Digikey, Notes, KiLib_Generator, Mouser, Arrow fields.
InvenTree IPN is now the only external reference in the schematic.
Parts:
- C25, C29, C30, C32, C33, C34, C35, C36, C39, C40, C41, C42, C43, C44, C46: KiLib_Generator SMD_2terminal_chip_molded -> (none); Notes 10% or 20% 35V Ceramic Capacitor X6S 0805 (2012 Metric) -> (none); Supplier https://www.digikey.ch/de/products/detail/samsung-electro-m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 -> (none)
- C26: KiLib_Generator capacitor/SMD/elec_round_polarized -> (none)
- C27: KiLib_Generator SMD_2terminal_chip_molded -> (none); Notes 10% 10V Ceramic Capacitor X5R -> (none); Supplier https://www.digikey.ch/de/products/detail/murata-electronic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 -> (none)
- C28, C45: Digikey 1276-1180-1-ND -> (none); KiLib_Generator SMD_2terminal_chip_molded -> (none); Notes 10% 16V Ceramic Capacitor X7R -> (none); Supplier https://www.digikey.ch/de/products/detail/samsung-electro-m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 -> (none)
- C31, C37: KiLib_Generator SMD_2terminal_chip_molded -> (none); Notes 1000 pF, 50 V -> (none); Supplier https://www.digikey.ch/de/products/detail/samsung-electro-m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 -> (none)
- C38: KiLib_Generator SMD_2terminal_chip_molded -> (none); Notes Capacitor, SP-Cap, 100u, 6.3V, 15mR ESR -> (none); Supplier https://www.digikey.ch/de/products/detail/panasonic-electro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 -> (none)
- F1: KiLib_Generator SMD_2terminal_chip_molded -> (none)
- J6: KiLib_Generator terminal_block/Phoenix -> (none); Supplier https://www.digikey.ch/de/products/detail/phoenix-contact/1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 -> (none)
- J7: Supplier https://www.digikey.ch/de/products/detail/w%C3%BCrth-elektr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 -> (none)
- L1: Notes 3.3µH Semi-Shielded Wirewound Inductor 7.8A 21mOhm Nonstand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 -> (none); Supplier https://www.digikey.ch/de/products/detail/bourns-inc/SRN604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 -> (none)
- Q6: IPN Q-001 -> (none); Supplier https://www.digikey.ch/de/products/detail/onsemi/FDS4435BZ/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 -> (none)
- R24: KiLib_Generator SMD_2terminal_chip_molded -> (none); Notes Resistor 2.2K 1% 63mW -> (none); Supplier https://www.digikey.ch/de/products/detail/stackpole-electro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 -> (none)
- R25: KiLib_Generator SMD_2terminal_chip_molded -> (none); Notes Resistor 20K 1% 63mW -> (none); Supplier https://www.digikey.ch/de/products/detail/stackpole-electro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 -> (none)
- R26: KiLib_Generator SMD_2terminal_chip_molded -> (none); Notes Resistor 12K 1% 63mW -> (none); Supplier https://www.digikey.ch/de/products/detail/stackpole-electro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 -> (none)
- R27: KiLib_Generator SMD_2terminal_chip_molded -> (none); Notes Resistor 10R 1% 63mW -> (none); Supplier https://www.digikey.ch/de/products/detail/stackpole-electro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 -> (none)
- U6: Supplier https://www.digikey.ch/de/products/detail/diodes-incorporat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 -> (none)
- U7: IPN U-001 -> (none); Supplier https://www.digikey.ch/de/products/detail/diodes-incorporat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 -> (none)

Commit message: feat: complete IPN assignment for all BOM parts
All components now have InvenTree IPN field.
Added IPN to granit library symbols (ASM1061, FDS4435BZ, AP64501).
Added Q-003 to 2N7002 instances.
Only TestPoints have no IPN (not purchaseable).
Parts:
- Q6: IPN (none) -> Q-001
- U7: IPN (none) -> U-001
Changed lines of the file:
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@@
+			)
+		)
+		(property "IPN" "U-001"
+			(at 142.24 127 0)
+			(hide yes)
+			(show_name no)
+			(do_not_autoplace no)
+			(effects
+				(font
+					(size 1.27 1.27)
+				)
 			)
 		)
@@
 			(at 93.98 44.45 0)
 			(hide yes)
+			(show_name no)
+			(do_not_autoplace no)
+			(effects
+				(font
+					(size 1.27 1.27)
+				)
+			)
+		)
+		(property "IPN" "Q-001"
+			(at 93.98 44.45 0)
+			(hide yes)

Commit message: feat: swap C26 footprint to CP_Elec_6.3x7.7 (easier to source on LCSC)
Parts:
- C26: footprint Capacitor_SMD:CP_Elec_6.3x5.8 -> Capacitor_SMD:CP_Elec_6.3x7.7
Changed lines of the file:
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@@
 			)
 		)
-		(property "Footprint" "Capacitor_SMD:CP_Elec_6.3x5.8"
+		(property "Footprint" "Capacitor_SMD:CP_Elec_6.3x7.7"
 			(at 119.0752 64.77 0)
 			(hide yes)
