File: latest/kicad/granit.kicad_pcb (KiCad board)
At the start: 4 copper layers, 92 x 99.5 mm, 120 parts, among them J1 USB_C_Receptacle_USB2.0_14P, J2 PCM12SMTR, J3 BM03B-SRSS-TB, J4 SATA_22pin, J6 12V Screw Terminal, J7 12V Barrel, J8 HR911130A, Q1 2N7002, Q2 FDS4435BZ, Q3 FDS4435BZ, Q4 2N7002, Q5 2N7002, Q6 FDS4435BZ, SW1 SW_Push, U1 USBLC6-2SC6, U2 74AHCT1G125, U3 ASM1061, U4 74AHCT1G32, U5 DS3231MZ, U6 NCP1117-3.3_SOT223, U7 AP64501SP-13, Y1 25MHz

Commit message: Deploying to gh-pages from @ laenzlinger/granit@f994fe32861f9e128897c0b4695d907eee013e28 🚀
Other:
- board text added: "CH000031"
Changed lines of the file:
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@@
+		)
+	)
+	(gr_text "CH000031"
+		(at 56.6 30.45 0)
+		(layer "F.SilkS")
+		(effects
+			(font
+				(size 0.8 0.8)
+				(thickness 0.15)
+			)
 		)
 	)
